Commit message: update

File: xacro/sick_wagen.xacro (robot description, xacro)
@@ -127,9 +127,9 @@
   <xacro:front_wheel_macro prefix="right_wheel" parent="base_floor" xyz="0.3 0.245 0" />
   <joint name="lidar_joint" type="fixed">
-    <parent link="base_floor" />
-    <child link="lidar_link" />
-    <origin xyz="0 0 0.25" rpy="0 0 0" />
-  </joint>
-  <link name="lidar_link">
+    <parent link="base_link" />
+    <child link="multiscan_link" />
+    <origin xyz="0 0 1.60" rpy="0 0 0" />
+  </joint>
+  <link name="multiscan_link">
     <visual>
       <geometry>
@@ -141,5 +141,5 @@
     <collision>
       <geometry>
-        <cylinder radius="0.030" length="0.086" />
+        <cylinder radius="0.0" length="0.086" />
       </geometry>
       <origin xyz="0 0 0" rpy="0 0 0" />
@@ -154,4 +154,54 @@
         izx="0" izy="0" izz="0.0001125" />
     </inertial>
+  </link>
+  <joint name="gps_joint" type="fixed">
+    <parent link="base_link" />
+    <child link="gps" />
+    <origin xyz="0.3 0 0.70" rpy="0 0 0" />
+  </joint>
+  <link name="gps">
+    <inertial>
+      <origin xyz="0 0 0" rpy="0 0 0" />
+      <mass value="0.10"/>
+      <inertia ixx="0.001" ixy="0.0" ixz="0.0" iyy="0.001" iyz="0.0" izz="0.001" />
+    </inertial>
+    <visual>
+      <origin xyz="0 0 0" rpy="0 0 0" />
+      <geometry>
+        <box size="0.10 0.10 0.030" />
+      </geometry>
+      <material name="green" />
+    </visual>
+    <collision>
+      <origin xyz="0 0 0" rpy="0 0 0" />
+      <geometry>
+        <box size="0.10 0.10 0.030" />
+      </geometry>
+    </collision>
+  </link>
+  <joint name="imu_joint" type="fixed">
+    <parent link="base_link" />
+    <child link="imu_link" />
+    <origin xyz="0.0 0 1.00" rpy="0 0 0" />
+  </joint>
+  <link name="imu_link">
+    <inertial>
+      <origin xyz="0 0 0" rpy="0 0 0" />
+      <mass value="0.10"/>
+      <inertia ixx="0.001" ixy="0.0" ixz="0.0" iyy="0.001" iyz="0.0" izz="0.001" />
+    </inertial>
+    <visual>
+      <origin xyz="0 0 0" rpy="0 0 0" />
+      <geometry>
+        <box size="0.050 0.050 0.030" />
+      </geometry>
+      <material name="green" />
+    </visual>
+    <collision>
+      <origin xyz="0 0 0" rpy="0 0 0" />
+      <geometry>
+        <box size="0.050 0.050 0.030" />
+      </geometry>
+    </collision>
   </link>
   <gazebo reference="lidar_link">

Commit message: update

File: xacro/sick_wagen.xacro (robot description, xacro)
@@ -1,4 +1,4 @@
 <?xml version="1.0"?>
-<robot name="dtw_robot" xmlns:xacro="http://ros.org/wiki/xacro">
+<robot xmlns:xacro="http://www.ros.org/wiki/xacro" name="whill_modelc">
   <material name="gray">
     <color rgba="0.5 0.5 0.5 1.0" />
@@ -14,83 +14,6 @@
   </material>
   <material name="black">
-    <color rgba="0.0 0.0 0.0 1.0" />
-  </material>
-  <!-- Rear wheel macro -->
-  <xacro:macro name="rear_wheel_macro" params="parent prefix xyz">
-    <joint name="${prefix}_joint" type="continuous">
-      <origin xyz="${xyz}" rpy="${radians(-90)} 0 0" />
-      <parent link="${parent}" />
-      <child link="${prefix}_link" />
-      <axis xyz="0 0 1" />
-    </joint>
-    <transmission name="${prefix}_trans" type="SimpleTransmission">
-      <type>transmission_interface/SimpleTransmission</type>
-      <actuator name="${prefix}_motor">
-        <mechanicalReduction>1</mechanicalReduction>
-      </actuator>
-      <joint name="${prefix}_joint">
-        <hardwareInterface>hardware_interface/VelocityJointInterface</hardwareInterface>
-      </joint>
-    </transmission>
-    <link name="${prefix}_link">
-      <inertial>
-        <origin xyz="0 0 0" rpy="0 0 0" />
-        <mass value="0.1" />
-        <inertia ixx="0.0001" ixy="0.0" ixz="0.0" iyy="0.0001" iyz="0.0" izz="0.0001" />
-      </inertial>
-      <visual>
-        <geometry>
-          <cylinder radius="0.1325" length="0.05" />
-        </geometry>
-        <material name="red" />
-      </visual>
-      <collision>
-        <geometry>
-          <cylinder radius="0.1325" length="0.05" />
-        </geometry>
-      </collision>
-    </link>
-    <gazebo reference="${prefix}_link">
-      <material>Gazebo/Red</material>
-      <mu1 value="3.5" />
-      <mu2 value="3.5" />
-      <kp value="10000" />
-      <kd value="10" />
-    </gazebo>
-  </xacro:macro>
-  <!-- Front wheel macro -->
-  <xacro:macro name="front_wheel_macro" params="parent prefix xyz">
-    <link name="front_${prefix}_link">
-      <collision>
-        <geometry>
-          <sphere radius="0.1325" />
-        </geometry>
-      </collision>
-      <visual>
-        <geometry>
-          <cylinder length="0.05" radius="0.1325" />
-        </geometry>
-        <material name="black" />
-      </visual>
-      <inertial>
-        <origin xyz="0 0 0" rpy="0 0 0" />
-        <mass value="1.0" />
-        <inertia ixx="1.0" ixy="0.0" ixz="0.0"
-          iyy="1.0" iyz="0.0"
-          izz="1.0" />
-      </inertial>
-    </link>
-    <joint name="front_${prefix}_joint" type="fixed">
-      <parent link="${parent}" />
-      <child link="front_${prefix}_link" />
-      <origin xyz="${xyz}" rpy="${radians(90)} 0 0" />
-      <axis xyz="0 0 1" />
-    </joint>
-    <gazebo reference="front_${prefix}_link">
-      <material>Gazebo/Black</material>
-      <mu1 value="0.01" />
-      <mu2 value="0.01" />
-    </gazebo>
-  </xacro:macro>
+    <color rgba="0.2 0.2 0.2 1.0" />
+  </material>
   <link name="base_link" />
   <joint name="base_body_joint" type="fixed">
@@ -108,5 +31,5 @@
       <origin xyz="0 0 0" rpy="0 0 0" />
       <geometry>
-        <box size="0.600 0.400 0.050" />
+        <box size="0.85 0.4 0.050" />
       </geometry>
       <material name="green" />
@@ -115,21 +38,144 @@
       <origin xyz="0 0 0" rpy="0 0 0" />
       <geometry>
-        <box size="0.600 0.400 0.050" />
-      </geometry>
-    </collision>
-  </link>
-  <gazebo reference="base_floor">
-    <material>Gazebo/Green</material>
-  </gazebo>
-  <xacro:rear_wheel_macro prefix="left_wheel" parent="base_floor" xyz="-0.3 0.245 0" />
-  <xacro:rear_wheel_macro prefix="right_wheel" parent="base_floor" xyz="-0.3 -0.245 0" />
-  <xacro:front_wheel_macro prefix="left_wheel" parent="base_floor" xyz="0.3 -0.245 0" />
-  <xacro:front_wheel_macro prefix="right_wheel" parent="base_floor" xyz="0.3 0.245 0" />
-  <joint name="lidar_joint" type="fixed">
-    <parent link="base_link" />
-    <child link="multiscan_link" />
-    <origin xyz="0 0 1.60" rpy="0 0 0" />
-  </joint>
-  <link name="multiscan_link">
+        <box size="0.85 0.4 0.050" />
+      </geometry>
+    </collision>
+  </link>
+  <link name="left_wheel_link">
+    <visual>
+      <geometry>
+        <cylinder length="0.05" radius="0.1325" />
+      </geometry>
+      <origin xyz="0 0 0" rpy="0 0 0" />
+      <material name="red" />
+    </visual>
+    <collision>
+      <geometry>
+        <cylinder length="0.05" radius="0.1325" />
+      </geometry>
+    </collision>
+    <inertial>
+      <origin xyz="0 0 0" />
+      <mass value="0.500" />
+      <inertia ixx="0.0013541667" ixy="0" ixz="0" iyy="0.0013541667" iyz="0" izz="0.0025" />
+    </inertial>
+  </link>
+  <joint name="leftWheel" type="continuous">
+    <parent link="base_floor" />
+    <child link="left_wheel_link" />
+    <origin xyz="-0.3 0.245 0" rpy="-1.57 0 0" />
+    <axis xyz="0 0 1" />
+  </joint>
+  <link name="right_wheel_link">
+    <collision>
+      <origin xyz="0 0 0" rpy="0 0 0" />
+      <geometry>
+        <cylinder length="0.05" radius="0.1325" />
+      </geometry>
+    </collision>
+    <visual>
+      <origin xyz="0 0 0" rpy="0 0 0" />
+      <geometry>
+        <cylinder length="0.05" radius="0.1325" />
+      </geometry>
+      <material name="red" />
+    </visual>
+    <inertial>
+      <origin xyz="0 0 0" />
+      <mass value="0.500" />
+      <inertia ixx="0.0013541667" ixy="0" ixz="0" iyy="0.0013541667" iyz="0" izz="0.0025" />
+    </inertial>
+  </link>
+  <joint name="rightWheel" type="continuous">
+    <parent link="base_floor" />
+    <child link="right_wheel_link" />
+    <origin xyz="-0.3 -0.245 0" rpy="1.57 0 0" />
+    <axis xyz="0 0 1" />
+  </joint>
+  <link name="frontwheel_left">
+    <collision>
+      <geometry>
+        <cylinder length="0.05" radius="0.1325" />
+      </geometry>
+    </collision>
+    <visual>
+      <geometry>
+        <cylinder length="0.05" radius="0.1325" />
+      </geometry>
+      <material name="red" />
+    </visual>
+    <inertial>
+      <origin xyz="0 0 0" rpy="0 0 0" />
+      <mass value="1.0" />
+      <inertia ixx="1.0" ixy="0.0" ixz="0.0"
+        iyy="1.0" iyz="0.0"
+        izz="1.0" />
+    </inertial>
+  </link>
+  <joint name="frontwheel_left_joint" type="fixed">
+    <parent link="base_floor" />
+    <child link="frontwheel_left" />
+    <origin xyz="0.3 -0.245 0" rpy="1.57 0 0" />
+    <axis xyz="0 0 1" />
+  </joint>
+  <link name="frontwheel_right">
+    <collision>
+      <geometry>
+        <cylinder length="0.05" radius="0.1325" />
+      </geometry>
+    </collision>
+    <visual>
+      <geometry>
+        <cylinder length="0.05" radius="0.1325" />
+      </geometry>
+      <material name="red" />
+    </visual>
+    <inertial>
+      <origin xyz="0 0 0" rpy="0 0 0" />
+      <mass value="1.0" />
+      <inertia ixx="1.0" ixy="0.0" ixz="0.0"
+        iyy="1.0" iyz="0.0"
+        izz="1.0" />
+    </inertial>
+  </link>
+  <joint name="frontwheel_right_joint" type="fixed">
+    <parent link="base_floor" />
+    <child link="frontwheel_right" />
+    <origin xyz="0.3 0.245 0" rpy="1.57 0 0" />
+    <axis xyz="0 0 -1" />
+  </joint>
+  <!-- tim_frame-->
+  <joint name="tim_frame_joint" type="fixed">
+    <parent link="base_link" />
+    <child link="tim_frame" />
+    <origin xyz="0.82 0 0.0" rpy="0 0 0" />
+  </joint>
+  <link name="tim_frame">
+    <inertial>
+      <origin xyz="0 0 0" rpy="0 0 0" />
+      <mass value="1.0" />
+      <inertia ixx="0.001" ixy="0.0" ixz="0.0" iyy="0.001" iyz="0.0" izz="0.001" />
+    </inertial>
+    <visual>
+      <origin xyz="0 0 0" rpy="0 0 0" />
+      <geometry>
+        <box size="0.125 0.66 0.050" />
+      </geometry>
+      <material name="black" />
+    </visual>
+    <collision>
+      <origin xyz="0 0 0" rpy="0 0 0" />
+      <geometry>
+        <box size="0.10 0.66 0.050" />
+      </geometry>
+    </collision>
+  </link>
+  <!-- Tim_R %%%%%%%%%%%%%%%%%%%%%%%%%%%%%%%%%%%%%%%%%%-->
+  <joint name="tim_joint_R" type="fixed">
+    <parent link="base_link" />
+    <child link="tim_link_R" />
+    <origin xyz="0.82 -0.29 0.075" rpy="0 0 -0.84806208" />
+  </joint>
+  <link name="tim_link_R">
     <visual>
       <geometry>
@@ -141,5 +187,5 @@
     <collision>
       <geometry>
-        <cylinder radius="0.0" length="0.086" />
+        <cylinder radius="0.030" length="0.086" />
       </geometry>
       <origin xyz="0 0 0" rpy="0 0 0" />
@@ -155,100 +201,171 @@
     </inertial>
   </link>
+  <!-- Tim_L %%%%%%%%%%%%%%%%%%%%%%%%%%%%%%%%%%%%%%%%%%-->
+  <joint name="tim_joint_L" type="fixed">
+    <parent link="base_link" />
+    <child link="tim_link_L" />
+    <origin xyz="0.82 0.29 0.075" rpy="0 0 0.84806208" /> <!--ベースリンクからの距離 -->
+  </joint>
+  <link name="tim_link_L">
+    <visual>
+      <geometry>
+        <cylinder radius="0.030" length="0.086" />
+      </geometry>
+      <origin xyz="0 0 0" rpy="0 0 0" />
+      <material name="blue" />
+    </visual>
+    <collision>
+      <geometry>
+        <cylinder radius="0.030" length="0.086" />
+      </geometry>
+      <origin xyz="0 0 0" rpy="0 0 0" />
+    </collision>
+    <inertial>
+      <origin xyz="0 0 0" rpy="0 0 0" />
+      <mass value="0.25" />
+      <inertia ixx="0.00021033333"
+        ixy="0" ixz="0"
+        iyx="0" iyy="0.00021033333"
+        iyz="0"
+        izx="0" izy="0" izz="0.0001125" />
+    </inertial>
+  </link>
+  <!-- laser %%%%%%%%%%%%%%%%%%%%%%%%%%%%%%%%%%%%%%%%%%-->
+  <joint name="laser_joint" type="fixed">
+    <parent link="base_link" />
+    <child link="laser_link" />
+    <origin xyz="0.82 0 0.075" rpy="0 0 0" /> <!--ベースリンクからの距離 -->
+  </joint>
+  <link name="laser_link">
+    <visual>
+      <geometry>
+        <cylinder radius="0.01" length="0.01" />
+      </geometry>
+      <origin xyz="0 0 0" rpy="0 0 0" />
+      <material name="blue" />
+    </visual>
+    <collision>
+      <geometry>
+        <cylinder radius="0.01" length="0.01" />
+      </geometry>
+      <origin xyz="0 0 0" rpy="0 0 0" />
+    </collision>
+    <inertial>
+      <origin xyz="0 0 0" rpy="0 0 0" />
+      <mass value="0.25" />
+      <inertia ixx="0.00021033333"
+        ixy="0" ixz="0"
+        iyx="0" iyy="0.00021033333"
+        iyz="0"
+        izx="0" izy="0" izz="0.0001125" />
+    </inertial>
+  </link>
+  <!-- multiscan %%%%%%%%%%%%%%%%%%%%%%%%%%%%%%%%%%%%%%%%%%-->
+  <joint name="multiscan_joint" type="fixed">
+    <parent link="base_link" />
+    <child link="multiscan_link" />
+    <origin xyz="-0.10 0 1.545" rpy="0 0 0" />
+  </joint>
+  <link name="multiscan_link">
+    <visual>
+      <geometry>
+        <cylinder radius="0.060" length="0.086" />
+      </geometry>
+      <origin xyz="0 0 0" rpy="0 0 0" />
+      <material name="blue" />
+    </visual>
+    <collision>
+      <geometry>
+        <cylinder radius="0.060" length="0.086" />
+      </geometry>
+      <origin xyz="0 0 0" rpy="0 0 0" />
+    </collision>
+    <inertial>
+      <origin xyz="0 0 0" rpy="0 0 0" />
+      <mass value="0.25" />
+      <inertia ixx="0.00021033333"
+        ixy="0" ixz="0"
+        iyx="0" iyy="0.00021033333"
+        iyz="0"
+        izx="0" izy="0" izz="0.0001125" />
+    </inertial>
+  </link>
+  <!-- imu %%%%%%%%%%%%%%%%%%%%%%%%%%%%%%%%%%%%%%%%%%-->
+  <joint name="imu_joint" type="fixed">
+    <parent link="base_link" />
+    <child link="imu_link" />
+    <origin xyz="-0.14 0 1.05" rpy="0 0 0" />
+  </joint>
+  <link name="imu_link">
+    <inertial>
+      <origin xyz="0 0 0" rpy="0 0 0" />
+      <mass value="1.0" />
+      <inertia ixx="0.001" ixy="0.0" ixz="0.0" iyy="0.001" iyz="0.0" izz="0.001" />
+    </inertial>
+    <visual>
+      <origin xyz="0 0 0" rpy="0 0 0" />
+      <geometry>
+        <box size="0.06 0.06 0.020" />
+      </geometry>
+      <material name="black" />
+    </visual>
+    <collision>
+      <origin xyz="0 0 0" rpy="0 0 0" />
+      <geometry>
+        <box size="0.10 0.66 0.050" />
+      </geometry>
+    </collision>
+  </link>
+  <!-- web camear %%%%%%%%%%%%%%%%%%%%%%%%%%%%%%%%%%%%%%%%%%-->
+  <joint name="camera_joint" type="fixed">
+    <parent link="base_link" />
+    <child link="camera_link" />
+    <origin xyz="-0.14 0 1.40" rpy="0 0 0" />
+  </joint>
+  <link name="camera_link">
+    <inertial>
+      <origin xyz="0 0 0" rpy="0 0 0" />
+      <mass value="1.0" />
+      <inertia ixx="0.001" ixy="0.0" ixz="0.0" iyy="0.001" iyz="0.0" izz="0.001" />
+    </inertial>
+    <visual>
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
Commit message: add pointcloud merge test

File: xacro/sick_wagen.xacro (robot description, xacro)
@@ -266,4 +266,6 @@
     <child link="multiscan_link" />
     <origin xyz="-0.10 0 1.545" rpy="0 0 0" />
+    <!-- 上下反転する場合 -->
+    <!-- <origin xyz="-0.10 0 1.545" rpy="3.14 0 0" /> -->
   </joint>
   <link name="multiscan_link">

Commit message: multiscanを上下逆転

File: xacro/sick_wagen.xacro (robot description, xacro)
@@ -265,7 +265,7 @@
     <parent link="base_link" />
     <child link="multiscan_link" />
-    <origin xyz="-0.10 0 1.545" rpy="0 0 0" />
+    <origin xyz="-0.10 0 1.42" rpy="0 0 0" />
     <!-- 上下反転する場合 -->
-    <!-- <origin xyz="-0.10 0 1.545" rpy="3.14 0 0" /> -->
+    <!-- <origin xyz="-0.10 0 1.42" rpy="3.14 0 0" /> -->
   </joint>
   <link name="multiscan_link">

Commit message: gennjyou

File: xacro/sick_wagen.xacro (robot description, xacro)
@@ -297,5 +297,5 @@
     <parent link="base_link" />
     <child link="imu_link" />
-    <origin xyz="-0.14 0 1.05" rpy="0 0 0" />
+    <origin xyz="0.47 0 0.26" rpy="0 0 0" />
   </joint>
   <link name="imu_link">
@@ -323,5 +323,5 @@
     <parent link="base_link" />
     <child link="camera_link" />
-    <origin xyz="-0.14 0 1.40" rpy="0 0 0" />
+    <origin xyz="-0.14 0 1.35" rpy="0 0 0" />
   </joint>
   <link name="camera_link">
@@ -349,5 +349,5 @@
     <parent link="base_link" />
     <child link="gps_link" />
-    <origin xyz="0.12 0.25 1.03" rpy="0 0 0" />
+    <origin xyz="-0.10 -0.15 1.42" rpy="0 0 0" />
   </joint>
   <link name="gps_link">
